File: blocky_breakout_pcb/arduino_headers.kicad_sch (KiCad schematic)
At the start: 4 parts, among them J4 Conn_01x08_Pin, J5 Conn_01x10_Pin, J6 Conn_01x06_Pin, J7 Conn_01x08_Pin

Commit message: Layout nearly finished, entering part numbers
Connections:
- net I2C0.SCL renamed I2C1.SCL
- net I2C0.SDA renamed I2C1.SDA
Changed lines of the file:
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@@
 		)
 	)
-	(label "I2C0.SDA"
+	(label "I2C1.SDA"
 		(at 182.88 74.93 0)
 		(effects
@@
 		)
 	)
-	(label "I2C0.SCL"
+	(label "I2C1.SCL"
 		(at 182.88 72.39 0)
 		(effects
@@
 		)
 	)
-	(hierarchical_label "{I2C0}"
+	(hierarchical_label "{I2C1}"
 		(shape output)
 		(at 199.39 66.04 0)
