File: blocky_breakout_pcb/dac.kicad_sch (KiCad schematic)
At the start: 5 parts, among them U8 MCP4728

Commit message: Layout nearly finished, entering part numbers
Parts:
- C27: MPN (none) -> CL05B104KP5NNNC
- C28: footprint Capacitor_SMD:C_0603_1608Metric -> Capacitor_SMD:C_0402_1005Metric; MPN (none) -> JMK105BBJ475MV-F
- R15, R16: MPN (none) -> RC0402FR-131KL
- U8: MPN (none) -> MCP4728T-E/UN
Connections:
- net DAC0: now reaches U8.6 (VOUTA)
- net DAC1: now reaches U8.7 (VOUTB)
- net DAC2: now reaches U8.8 (VOUTC)
- net DAC3: now reaches U8.9 (VOUTD)
- net I2C1.SCL renamed I2C0.SCL
- net I2C1.SDA renamed I2C0.SDA
Changed lines of the file:
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@@
 	(wire
 		(pts
+			(xy 170.18 97.79) (xy 180.34 97.79)
+		)
+		(stroke
+			(width 0)
+			(type default)
+		)
+	)
+	(wire
+		(pts
 			(xy 158.75 85.09) (xy 158.75 83.82)
 		)
@@
 	(wire
 		(pts
+			(xy 170.18 100.33) (xy 180.34 100.33)
+		)
+		(stroke
+			(width 0)
+			(type default)
+		)
+	)
+	(wire
+		(pts
 			(xy 127 92.71) (xy 127 97.79)
 		)
@@
 		)
 	)
+	(wire
+		(pts
+			(xy 170.18 102.87) (xy 180.34 102.87)
+		)
+		(stroke
+			(width 0)
+			(type default)
+		)
+	)
 	(bus
 		(pts
@@
 	(wire
 		(pts
+			(xy 170.18 95.25) (xy 180.34 95.25)
+		)
+		(stroke
+			(width 0)
+			(type default)
+		)
+	)
+	(wire
+		(pts
 			(xy 154.94 113.03) (xy 154.94 107.95)
 		)
@@
 		)
 	)
-	(label "I2C1.SDA"
+	(label "I2C0.SDA"
 		(at 138.43 97.79 180)
 		(effects
@@
 		)
 	)
-	(label "I2C1.SCL"
+	(label "I2C0.SCL"
 		(at 138.43 95.25 180)
 		(effects
@@
 		)
 	)
-	(hierarchical_label "{I2C1}"
+	(hierarchical_label "{I2C0}"
 		(shape output)
 		(at 110.49 88.9 180)
@@
 		)
 	)
+	(hierarchical_label "DAC3"
+		(shape output)
+		(at 180.34 102.87 0)
+		(effects
+			(font
+				(size 1.27 1.27)
+			)
+			(justify left)
+		)
+	)
+	(hierarchical_label "DAC2"
+		(shape output)
+		(at 180.34 100.33 0)
+		(effects
+			(font
+				(size 1.27 1.27)
+			)
+			(justify left)
+		)
+	)
+	(hierarchical_label "DAC1"
+		(shape output)
+		(at 180.34 97.79 0)
+		(effects
+			(font
+				(size 1.27 1.27)
+			)
+			(justify left)
+		)
+	)
+	(hierarchical_label "DAC0"
+		(shape output)
+		(at 180.34 95.25 0)
+		(effects
+			(font
+				(size 1.27 1.27)
+			)
+			(justify left)
+		)
+	)
 	(symbol
 		(lib_id "Device:R_Small_US")
@@
 		)
 		(property "Sim.Type" ""
+			(at 127 90.17 0)
+			(effects
+				(font
+					(size 1.27 1.27)
+				)
+				(hide yes)
+			)
+		)
+		(property "MPN" "RC0402FR-131KL"
 			(at 127 90.17 0)
 			(effects
@@
 			)
 		)
+		(property "MPN" "CL05B104KP5NNNC"
+			(at 151.13 81.28 0)
+			(effects
+				(font
+					(size 1.27 1.27)
+				)
+				(hide yes)
+			)
+		)
 		(pin "1"
 		)
@@
 			)
 		)
-		(property "Footprint" "Capacitor_SMD:C_0603_1608Metric"
+		(property "Footprint" "Capacitor_SMD:C_0402_1005Metric"
 			(at 158.75 81.28 0)
 			(effects
@@
 		)
 		(property "Sim.Type" ""
+			(at 158.75 81.28 0)
+			(effects
+				(font
+					(size 1.27 1.27)
+				)
+				(hide yes)
+			)
+		)
+		(property "MPN" "JMK105BBJ475MV-F"
 			(at 158.75 81.28 0)
 			(effects
@@
 			)
 		)
+		(property "MPN" "RC0402FR-131KL"
+			(at 120.65 90.17 0)
+			(effects
+				(font
+					(size 1.27 1.27)
+				)
+				(hide yes)
+			)
+		)
 		(pin "2"
 		)
@@
 			(at 154.94 97.79 0)
 			(effects
+				(font
+					(size 1.27 1.27)
+				)
+				(hide yes)
+			)
+		)
+		(property "MPN" "MCP4728T-E/UN"
+			(at 154.94 97.79 0)
+			(effects
