File: blocky_breakout_pcb/relay.kicad_sch (KiCad schematic)
At the start: 5 parts, among them J10 Conn_01x02_Pin, K1 EE2-3TNUH, Q1 DMG1012TQ-7

Commit message: Layout nearly finished, entering part numbers
Parts:
- R14: MPN (none) -> RC0402FR-131KL
Changed lines of the file:
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@@
+			)
+		)
+		(property "MPN" "RC0402FR-131KL"
+			(at 138.43 107.95 0)
+			(effects
+				(font
+					(size 1.27 1.27)
+				)
+				(hide yes)
 			)
 		)
