File: blocky_breakout_pcb/rpi_header.kicad_sch (KiCad schematic)
At the start: 1 part, among them J1 Raspberry_Pi_4

Commit message: Layout nearly finished, entering part numbers
Connections:
- net GPIO24: now reaches J1.18 (GPIO24/SDIO_DAT0)
- net GPIO25: now reaches J1.22 (GPIO25/SDIO_DAT1)
- net GPIO16: no longer names the net of J1.36 (GPIO16/SPI1_~{CE2})
- net GPIO17: no longer names the net of J1.11 (GPIO17/SPI1_~{CE1})
Changed lines of the file:
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@@
-	)
-	(no_connect
-		(at 118.11 113.03)
 	)
 	(no_connect
@@
 	)
 	(no_connect
-		(at 118.11 110.49)
+		(at 118.11 100.33)
 	)
 	(no_connect
-		(at 118.11 100.33)
+		(at 118.11 87.63)
 	)
 	(no_connect
@@
 	(no_connect
 		(at 184.15 105.41)
+	)
+	(no_connect
+		(at 118.11 90.17)
 	)
 	(no_connect
@@
 	(wire
 		(pts
-			(xy 113.03 87.63) (xy 118.11 87.63)
+			(xy 113.03 113.03) (xy 118.11 113.03)
 		)
 		(stroke
@@
 	(wire
 		(pts
-			(xy 113.03 90.17) (xy 118.11 90.17)
+			(xy 113.03 110.49) (xy 118.11 110.49)
 		)
 		(stroke
@@
 		)
 	)
-	(hierarchical_label "GPIO16"
+	(hierarchical_label "GPIO25"
 		(shape output)
-		(at 113.03 87.63 180)
+		(at 113.03 113.03 180)
 		(effects
 			(font
@@
 		)
 	)
-	(hierarchical_label "GPIO17"
+	(hierarchical_label "GPIO24"
 		(shape bidirectional)
-		(at 113.03 90.17 180)
+		(at 113.03 110.49 180)
 		(effects
 			(font
