File: blocky_breakout_pcb/rp2350.kicad_sch (KiCad schematic)
At the start: 47 parts, among them J2 USB_C_Receptacle_USB2.0_16P, J3 Conn_01x14_Pin, J9 Conn_01x03_Pin, SW1 SW_Push, SW2 SW_DIP_x04, U1 W25Q32JVSS, U2 NUP2202, U3 RP2350, U4 LM4040C33FTA, Y1 12Mhz

Commit message: Layout nearly finished, entering part numbers
Parts:
- C1: MPN (none) -> JMK105BJ105KV-F
- C10, C11, C12, C13, C3, C4, C5, C7, C8, C9: MPN (none) -> CL05B104KP5NNNC
- C14, C17, C6: footprint Capacitor_SMD:C_0603_1608Metric -> Capacitor_SMD:C_0402_1005Metric; MPN (none) -> JMK105BBJ475MV-F
- C15, C16: MPN (none) -> JMK105BBJ475MV-F
- C2: value 10nF -> 100nF; MPN (none) -> CL05B104KP5NNNC
- J9: footprint Connector_PinHeader_2.54mm:PinHeader_1x03_P2.54mm_Horizontal -> Connector_PinHeader_2.54mm:PinHeader_1x03_P2.54mm_Vertical
- R10, R18, R19, R2, R20, R5, R7: MPN (none) -> RC0402FR-131KL
- R4, R8, R9: MPN (none) -> RC0402FR-1327RL
- Y1: footprint Crystal:Crystal_SMD_Abracon_ABM8AIG-4Pin_3.2x2.5mm -> X_Abracon:Crystal_SMD_Abracon_ABM8-272-T3-4Pin_3.2x2.5mm; MPN ABM8AIG-12.000MHZ-12-2Z-T3 -> ABM8-272-T3
Connections:
- net D2: now also U3.8 (GPIO10); no longer U3.40 (GPIO32)
- net D3: now also U3.9 (GPIO11); no longer U3.42 (GPIO33)
- net D4: now also U3.11 (GPIO12); no longer U3.43 (GPIO34)
- net D5: now also U3.12 (GPIO13); no longer U3.44 (GPIO35)
- net D6: now also U3.13 (GPIO14); no longer U3.45 (GPIO36)
- net D7: now also U3.14 (GPIO15); no longer U3.46 (GPIO37)
- net D8: now also U3.16 (GPIO16); no longer U3.47 (GPIO38)
- net D9: now also U3.17 (GPIO17); no longer U3.48 (GPIO39)
- net GPIO26: now also J3.8 (Pin_8); no longer J3.6 (Pin_6)
- net GPIO27: now also J3.9 (Pin_9); no longer J3.7 (Pin_7)
- net GPIO28: now also J3.3 (Pin_3); no longer J3.8 (Pin_8)
- net GPIO29: now also J3.4 (Pin_4); no longer J3.9 (Pin_9)
- net GPIO30: now also J3.5 (Pin_5); no longer J3.10 (Pin_10)
- net GPIO31: now also J3.6 (Pin_6); no longer J3.11 (Pin_11)
- net GPIO46: now also J3.1 (Pin_1); no longer J3.12 (Pin_12)
- net GPIO47: now also J3.2 (Pin_2); no longer J3.13 (Pin_13)
- net GPIO6: no longer J3.1 (Pin_1)
- net GPIO7: no longer J3.2 (Pin_2)
- net I2C0.SCL: now also U3.2 (GPIO5); no longer U3.7 (GPIO9)
- net I2C0.SDA: now also U3.1 (GPIO4); no longer U3.6 (GPIO8)
- net I2C1.SCL: now also U3.23 (GPIO23); no longer U3.9 (GPIO11)
- net I2C1.SDA: now also U3.22 (GPIO22); no longer U3.8 (GPIO10)
- net SPI0.CS: now also U3.21 (GPIO21); no longer U3.2 (GPIO5)
- net SPI0.MISO: now also U3.20 (GPIO20); no longer U3.1 (GPIO4)
- net SPI0.MOSI: now also U3.19 (GPIO19); no longer U3.80 (GPIO3)
- net SPI0.SCK: now also U3.18 (GPIO18); no longer U3.79 (GPIO2)
- net UART1_RX: now also U3.7 (GPIO9); no longer U3.21 (GPIO21)
- net UART1_TX: now also U3.6 (GPIO8); no longer U3.20 (GPIO20)
- net GPIO12 renamed GPIO39
- net GPIO39: now also U3.48 (GPIO39); no longer U3.11 (GPIO12)
- net GPIO13 renamed GPIO38
- net GPIO38: now also U3.47 (GPIO38); no longer U3.12 (GPIO13)
- net GPIO14 renamed GPIO37
- net GPIO37: now also U3.46 (GPIO37); no longer U3.13 (GPIO14)
- net GPIO15 renamed GPIO36
- net GPIO36: now also U3.45 (GPIO36); no longer U3.14 (GPIO15)
- net GPIO16 renamed GPIO33
- net GPIO33: now also U3.42 (GPIO33); no longer U3.16 (GPIO16)
- net GPIO17 renamed GPIO34
- net GPIO34: now also U3.43 (GPIO34); no longer U3.17 (GPIO17)
- net GPIO18 renamed GPIO35
- net GPIO35: now also U3.44 (GPIO35); no longer U3.18 (GPIO18)
- removed net GPIO19: J3.3 (Pin_3), U3.19 (GPIO19)
- removed net GPIO22: J3.5 (Pin_5), U3.22 (GPIO22)
- removed net GPIO23: J3.4 (Pin_4), U3.23 (GPIO23)
- new net DAC0: J3.10 (Pin_10)
- new net DAC1: J3.11 (Pin_11)
- new net DAC2: J3.12 (Pin_12)
- new net DAC3: J3.13 (Pin_13)
- new net GPIO32: J3.7 (Pin_7), U3.40 (GPIO32)

Commit message: Added some docs, worked on routing.
Parts:
- added R21: 10k, Resistor_SMD:R_0402_1005Metric, symbol Device:R_Small_US
- added R22: 1k, Resistor_SMD:R_0402_1005Metric, symbol Device:R_Small_US
- added SW3: SW_Push, Button_Switch_SMD:SW_SPST_PTS647_Sx38, symbol Switch:SW_Push
- R5: now not fitted
- U3: MPN (none) -> RP2350B
Connections:
- net +1V1: now also L1.1; no longer L1.2
- net +3V3: now also R21.2
- net GND: now also R22.1
- net QSPI_~{SS}: now also R21.1
- net VREF_LX: now also L1.2; no longer L1.1
- net at R5.1, R6.2, U3.35 (RUN): now also SW3.2
- new net: R22.2, SW3.1
Other:
- moved on the sheet: L1, R6
