File: pcb/dac.kicad_sch (KiCad schematic)
At the start: 5 parts, among them U8 MCP4728

Commit message: R0.1 released
Parts:
- renumbered C27 to C29, C28 to C30, R15 to R19, R16 to R20, U8 to U9
Changed lines of the file:
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@@
 		(on_board yes)
 		(dnp no)
-		(property "Reference" "R16"
+		(property "Reference" "R20"
 			(at 124.079 88.9 0)
 			(effects
@@
 			(project "blocky_breakout_pcb"
 				(path "/deaf739e-0e27-4f2f-890a-6dd284a38e9f/03b50f7c-c1dd-4d8d-b088-fdeb50ef567a"
-					(reference "R16")
+					(reference "R20")
 					(unit 1)
 				)
@@
 		(dnp no)
 		(fields_autoplaced yes)
-		(property "Reference" "#PWR054"
+		(property "Reference" "#PWR063"
 			(at 158.75 91.44 0)
 			(effects
@@
 			(project "blocky_breakout_pcb"
 				(path "/deaf739e-0e27-4f2f-890a-6dd284a38e9f/03b50f7c-c1dd-4d8d-b088-fdeb50ef567a"
-					(reference "#PWR054")
+					(reference "#PWR063")
 					(unit 1)
 				)
@@
 		(dnp no)
 		(fields_autoplaced yes)
-		(property "Reference" "#PWR053"
+		(property "Reference" "#PWR062"
 			(at 151.13 91.44 0)
 			(effects
@@
 			(project "blocky_breakout_pcb"
 				(path "/deaf739e-0e27-4f2f-890a-6dd284a38e9f/03b50f7c-c1dd-4d8d-b088-fdeb50ef567a"
-					(reference "#PWR053")
+					(reference "#PWR062")
 					(unit 1)
 				)
@@
 		(on_board yes)
 		(dnp no)
-		(property "Reference" "C27"
+		(property "Reference" "C29"
 			(at 148.844 80.2578 0)
 			(effects
@@
 			(project "blocky_breakout_pcb"
 				(path "/deaf739e-0e27-4f2f-890a-6dd284a38e9f/03b50f7c-c1dd-4d8d-b088-fdeb50ef567a"
-					(reference "C27")
+					(reference "C29")
 					(unit 1)
 				)
@@
 		(dnp no)
 		(fields_autoplaced yes)
-		(property "Reference" "C28"
+		(property "Reference" "C30"
 			(at 161.29 80.0162 0)
 			(effects
@@
 			(project "blocky_breakout_pcb"
 				(path "/deaf739e-0e27-4f2f-890a-6dd284a38e9f/03b50f7c-c1dd-4d8d-b088-fdeb50ef567a"
-					(reference "C28")
+					(reference "C30")
 					(unit 1)
 				)
@@
 		(on_board yes)
 		(dnp no)
-		(property "Reference" "R15"
+		(property "Reference" "R19"
 			(at 117.729 88.9 0)
 			(effects
@@
 			(project "blocky_breakout_pcb"
 				(path "/deaf739e-0e27-4f2f-890a-6dd284a38e9f/03b50f7c-c1dd-4d8d-b088-fdeb50ef567a"
-					(reference "R15")
+					(reference "R19")
 					(unit 1)
 				)
@@
 		(dnp no)
 		(fields_autoplaced yes)
-		(property "Reference" "#PWR055"
+		(property "Reference" "#PWR064"
 			(at 154.94 119.38 0)
 			(effects
@@
 			(project "blocky_breakout_pcb"
 				(path "/deaf739e-0e27-4f2f-890a-6dd284a38e9f/03b50f7c-c1dd-4d8d-b088-fdeb50ef567a"
-					(reference "#PWR055")
+					(reference "#PWR064")
 					(unit 1)
 				)
@@
 		(on_board yes)
 		(dnp no)
-		(property "Reference" "#PWR052"
+		(property "Reference" "#PWR061"
 			(at 120.65 85.09 0)
 			(effects
@@
 			(project "blocky_breakout_pcb"
 				(path "/deaf739e-0e27-4f2f-890a-6dd284a38e9f/03b50f7c-c1dd-4d8d-b088-fdeb50ef567a"
-					(reference "#PWR052")
+					(reference "#PWR061")
 					(unit 1)
 				)
@@
 		(on_board yes)
 		(dnp no)
-		(property "Reference" "#PWR051"
+		(property "Reference" "#PWR060"
 			(at 154.94 80.01 0)
 			(effects
@@
 			(project "blocky_breakout_pcb"
 				(path "/deaf739e-0e27-4f2f-890a-6dd284a38e9f/03b50f7c-c1dd-4d8d-b088-fdeb50ef567a"
-					(reference "#PWR051")
+					(reference "#PWR060")
 					(unit 1)
 				)
@@
 		(on_board yes)
 		(dnp no)
-		(property "Reference" "U8"
+		(property "Reference" "U9"
 			(at 159.004 89.916 0)
 			(effects
@@
 			(project "blocky_breakout_pcb"
 				(path "/deaf739e-0e27-4f2f-890a-6dd284a38e9f/03b50f7c-c1dd-4d8d-b088-fdeb50ef567a"
-					(reference "U8")
-					(unit 1)
-				)
+					(reference "U9")
+					(unit 1)
+				)
