File: pcb/pmic.kicad_sch (KiCad schematic)
At the start: 19 parts, among them U5 LM66100DCK, U6 AOZ1280CI, U7 LM66100DCK, U9 TCR2EE11

Commit message: R0.1 released
Parts:
- renumbered C25 to C22, C26 to C23, C22 to C24, C23 to C25, C24 to C26, C29 to C27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
