File: pcb/relay.kicad_sch (KiCad schematic)
At the start: 5 parts, among them J10 Conn_01x02_Pin, K1 EE2-3TNUH, Q1 DMG1012TQ-7

Commit message: Added gerbers, added 2x3 Arduino header.
Parts:
- D2: MPN (none) -> 1N4148WT
- J10: MPN (none) -> S2B-XH-A
Changed lines of the file:
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@@
+			)
+		)
+		(property "MPN" "1N4148WT"
+			(at 138.43 80.01 90)
+			(effects
+				(font
+					(size 1.27 1.27)
+				)
+				(hide yes)
 			)
 		)
@@
 			(at 195.58 77.47 0)
 			(effects
+				(font
+					(size 1.27 1.27)
+				)
+				(hide yes)
+			)
+		)
+		(property "MPN" "S2B-XH-A"
+			(at 195.58 77.47 0)
+			(effects

Commit message: R0.1 released
Parts:
- removed J10: Conn_01x02_Pin, Connector_JST:JST_XH_S2B-XH-A-1_1x02_P2.50mm_Horizontal, symbol Connector:Conn_01x02_Pin
- removed K1: EE2-3TNUH, Relay_SMD:Relay_DPDT_Kemet_EE2_NU, symbol Relay:EE2-3NU
- added J10: Conn_01x03_Pin, Connector_JST:JST_XH_S3B-XH-A-1_1x03_P2.50mm_Horizontal, symbol Connector:Conn_01x03_Pin
- added K1: EE2-3NUH, Relay_SMD:Relay_DPDT_Kemet_EE2_NUH, symbol Relay:EE2-3NUH
- D5: renamed from D2; value 1N4148WT -> BAT54XV2T1G; MPN 1N4148WT -> BAT54XV2T1G
- renumbered R14 to R21
Connections:
- net +3V3: now also K1.1
- net at D5.2 (A), Q1.3 (D): now also K1.12
- new net: J10.1 (Pin_1), K1.10
- new net: J10.3 (Pin_3), K1.8
- new net: J10.2 (Pin_2), K1.9
